File: EAGLE_files/Team_14_PCB_Ver4.5.brd (EAGLE design)
At the start: 36.3 x 46 mm, 16 parts, among them Y2 CSTCE16M0V53-R0 16MHZ

Commit message: Pre-print update
Updated board with final fixes before printing
Parts:
- removed R5, R6: 4.7k, SmartPrj:R0603-ROUND
- added R7, R8: 4.7k, SmartPrj:R0603-ROUND
Connections:
- removed net N$3: COLOR_HEADER.4, R5.1
- removed net N$4: COLOR_HEADER.5, R6.1
- net +5V: now also R7.1, R8.1; no longer USB_SERIAL_HEADER.3
- net SDA_5V: now also COLOR_HEADER.5, R8.2; no longer R6.2
- net SDA_5V1: now also COLOR_HEADER.4, R7.2; no longer R5.2
Routing:
- net GND: track 115.3 -> 0.00 mm, vias 0 -> 14
- net SDA_5V1: track 3.58 -> 18.6 mm
- net SDA_5V: track 4.32 -> 19.0 mm
- net N$4: track 8.39 -> 0.00 mm
- net +5V: track 69.7 -> 77.9 mm
- net N$3: track 4.08 -> 0.00 mm
